Commit message: full model + gazebo launch

File: src/drone/description/robot.urdf.xacro (robot description, xacro)
@@ -2,3 +2,4 @@
 <robot xmlns:xacro="http://www.ros.org/wiki/xacro"  name="robot">
     <xacro:include filename="robot_core.xacro" />
+    <xacro:include filename="gazebo_control.xacro"/>
 </robot>

File: src/drone/description/robot_core.xacro (robot description, xacro)
@@ -30,4 +30,127 @@
             </geometry>
         </collision>
+        <xacro:inertial_box mass="2.5" x="0.14" y="0.725" z="0.14">
+            <origin xyz="0 0 0" rpy="${pi/2} 0 0" />
+        </xacro:inertial_box>
+    </link>
+    <!-- Prop 1 LINK -->
+    <joint name="prop1_joint" type="continuous">
+        <parent link="chassis"/>
+        <child link="prop1"/>
+        <origin xyz="0.340 -0.2495 0.04"/>
+        <axis xyz = "0 0 1"/>
+    </joint>
+    <link
+        name="prop1">
+        <visual>
+        <origin xyz="-0.47 0.155 -0.22" rpy="${pi/2} 0 0" />
+        <geometry>
+            <mesh filename="file://$(find drone)/meshes/prop1.stl" scale="0.001 0.001 0.001"/>
+        </geometry>
+        <material
+            name="">
+            <color
+            rgba="0.752941176470588 0.752941176470588 0.752941176470588 1" />
+        </material>
+        </visual>
+        <collision>
+            <origin xyz="-0.47 0.155 -0.22" rpy="${pi/2} 0 0" />
+            <geometry>
+                <mesh filename="file://$(find drone)/meshes/prop1.stl" scale="0.001 0.001 0.001"/>
+            </geometry>
+        </collision>
+        <xacro:inertial_cylinder mass="0.125" radius="0.20" length="0.02">
+            <origin xyz="-0.47 0.155 -0.22" rpy="${pi/2} 0 0" />
+        </xacro:inertial_cylinder>
+    </link>
+     <!-- Prop 2 LINK -->
+    <joint name="prop2_joint" type="continuous">
+        <parent link="chassis"/>
+        <child link="prop2"/>
+        <origin xyz="-0.340 -0.2495 0.04"/>
+        <axis xyz = "0 0 1"/>
+    </joint>
+    <link
+        name="prop2">
+        <visual>
+        <origin xyz="-0.47 0.155 -0.22" rpy="${pi/2} 0 0" />
+        <geometry>
+            <mesh filename="file://$(find drone)/meshes/prop1.stl" scale="0.001 0.001 0.001"/>
+        </geometry>
+        <material
+            name="">
+            <color
+            rgba="0.752941176470588 0.752941176470588 0.752941176470588 1" />
+        </material>
+        </visual>
+        <collision>
+            <origin xyz="-0.47 0.155 -0.22" rpy="${pi/2} 0 0" />
+            <geometry>
+                <mesh filename="file://$(find drone)/meshes/prop1.stl" scale="0.001 0.001 0.001"/>
+            </geometry>
+        </collision>
+        <xacro:inertial_cylinder mass="0.125" radius="0.20" length="0.02">
+            <origin xyz="-0.47 0.155 -0.22" rpy="${pi/2} 0 0" />
+        </xacro:inertial_cylinder>
+    </link>
+     <!-- Prop 3 LINK -->
+    <joint name="prop3_joint" type="continuous">
+        <parent link="chassis"/>
+        <child link="prop3"/>
+        <origin xyz="0.340 0.2495 0.04"/>
+        <axis xyz = "0 0 1"/>
+    </joint>
+    <link
+        name="prop3">
+        <visual>
+        <origin xyz="-0.47 0.155 -0.22" rpy="${pi/2} 0 0" />
+        <geometry>
+            <mesh filename="file://$(find drone)/meshes/prop1.stl" scale="0.001 0.001 0.001"/>
+        </geometry>
+        <material
+            name="">
+            <color
+            rgba="0.752941176470588 0.752941176470588 0.752941176470588 1" />
+        </material>
+        </visual>
+        <collision>
+            <origin xyz="-0.47 0.155 -0.22" rpy="${pi/2} 0 0" />
+            <geometry>
+                <mesh filename="file://$(find drone)/meshes/prop1.stl" scale="0.001 0.001 0.001"/>
+            </geometry>
+        </collision>
+        <xacro:inertial_cylinder mass="0.125" radius="0.20" length="0.02">
+            <origin xyz="-0.47 0.155 -0.22" rpy="${pi/2} 0 0" />
+        </xacro:inertial_cylinder>
+    </link>
+    <!-- Prop 4 LINK -->
+    <joint name="prop4_joint" type="continuous">
+        <parent link="chassis"/>
+        <child link="prop4"/>
+        <origin xyz="-0.340 0.2495 0.04"/>
+        <axis xyz = "0 0 1"/>
+    </joint>
+    <link
+        name="prop4">
+        <visual>
+        <origin xyz="-0.47 0.155 -0.22" rpy="${pi/2} 0 0" />
+        <geometry>
+            <mesh filename="file://$(find drone)/meshes/prop1.stl" scale="0.001 0.001 0.001"/>
+        </geometry>
+        <material
+            name="">
+            <color
+            rgba="0.752941176470588 0.752941176470588 0.752941176470588 1" />
+        </material>
+        </visual>
+        <collision>
+            <origin xyz="-0.47 0.155 -0.22" rpy="${pi/2} 0 0" />
+            <geometry>
+                <mesh filename="file://$(find drone)/meshes/prop1.stl" scale="0.001 0.001 0.001"/>
+            </geometry>
+        </collision>
+        <xacro:inertial_cylinder mass="0.125" radius="0.20" length="0.02">
+            <origin xyz="-0.47 0.155 -0.22" rpy="${pi/2} 0 0" />
+        </xacro:inertial_cylinder>
     </link>
 </robot>
